File: kraky.kicad_pcb (KiCad board)
At the start: 4 copper layers, 36 parts, among them J1 PINHD_1x10_Female, J2 JST_02, Q1 2N3904, SW1 Push_Button, SW2 Push_Button, SW3 Push_Button, SW4 Push_Button, SW5 SW_Nidec_CAS-120A1, U1 TP4056-42-ESOP8, U3 RFM98W-433S2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

Commit message: updated, read readme
Parts:
- removed A1: ESP32_DevKit_V1_DOIT_36GPIOs, PCM_SL_Development_Boards:DOIT_ESP32_DEVKIT_36Pins
- added C5: 100nF, Capacitor_THT:C_Axial_L3.8mm_D2.6mm_P7.50mm_Horizontal, F.Cu at (124.5, 122.8)
- added U2: ~, esp32-s3:esp32-s3, F.Cu at (144.5, 112.5)
- added U4: MPU6050, PCM_SL_Breakout_Boards:MPU6050_Breakout, F.Cu at (161.5, 119.5)
- C1, C10, C2, C3, C4, C6, C7, C8: footprint Capacitor_SMD:C_0805_2012Metric -> Capacitor_THT:C_Axial_L3.8mm_D2.6mm_P7.50mm_Horizontal
- PS1: footprint Converter_DCDC:Converter_DCDC_XP_POWER-IAxxxxD_THT -> Converter_DCDC:step up kraky
- R1, R2, R3, R4, R5, R6, R9: footprint Resistor_SMD:R_0805_2012Metric_Pad1.20x1.40mm_HandSolder -> Resistor_THT:R_Axial_DIN0204_L3.6mm_D1.6mm_P5.08mm_Horizontal
- SW5: footprint Button_Switch_SMD:Nidec_Copal_CAS-120A -> Button_Switch_THT:SW_Slide_SPDT_Angled_CK_OS102011MA1Q
- moved C4 20.3 mm to (161.4, 68.4)
- moved U6 20.3 mm to (167.0, 62.5)
- moved R4 14.8 mm to (169.0, 143.5)
- moved R5 13.0 mm to (178.0, 148.5)
- moved R9 10.5 mm to (109.0, 147.0)
- moved U3 9.13 mm to (167.8, 82.1)
- moved C8 9.13 mm to (163.9, 83.0)
- moved R3 7.52 mm to (183.0, 130.0)
- moved PS1 7.00 mm to (118.0, 130.0)
- moved C1 6.35 mm to (184.5, 64.2)
- moved R6 6.01 mm to (178.0, 124.5)
- moved SW1 5.89 mm to (163.2, 134.2)
- moved SW2 5.89 mm to (172.8, 139.2)
- moved SW4 5.89 mm to (182.2, 134.2)
- moved SW3 5.89 mm to (172.8, 128.8)
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Connections:
- A2 pad 2: Net-(A1-GND) -> Net-(A2-GND)
- BZ1 pad 2: Net-(A1-GND) -> Net-(Brd1-GND)
- Brd1 pad 1: Net-(A1-GND) -> Net-(Brd1-GND)
- Brd1 pad 2: Net-(A1-5V) -> Net-(Brd1-VCC)
- C10 pad 1: Net-(A1-5V) -> Net-(Brd1-GND)
- C10 pad 2: Net-(A1-GND) -> Net-(PS1--Vin)
- C2 pad 1: Net-(A1-GND) -> Net-(Brd1-GND)
- C2 pad 2: Net-(A1-VIN) -> Net-(Brd1-VCC)
- C3 pad 1: Net-(A1-GND) -> Net-(PS1--Vin)
- C3 pad 2: Net-(A1-5V) -> Net-(Brd1-VCC)
- C4 pad 2: Net-(A1-GND) -> Net-(Brd1-GND)
- C6 pad 2: Net-(A1-GND) -> Net-(Brd1-GND)
- C7 pad 1: Net-(A1-GND) -> Net-(A2-VS)
- C7 pad 2: Net-(A2-VS) -> Net-(Brd1-GND)
- C8 pad 1: Net-(A2-VS) -> Net-(Brd1-GND)
- C8 pad 2: Net-(A1-GND) -> Net-(A2-VS)
- D1 pad 1: Net-(A1-GND) -> Net-(PS1--Vin)
- IRLED1 pad 1: Net-(A1-GND) -> Net-(A2-GND)
- J1 pad 1: Net-(A1-ADC2_CH4/D13) -> Net-(A2-VS)
- J1 pad 10: Net-(A1-GND) -> Net-(U2-GPIO17)
- J1 pad 2: Net-(A1-ADC2_CH6/D14) -> Net-(Brd1-GND)
- J1 pad 3: Net-(A1-ADC2_CH7/D27) -> Net-(Brd1-GND)
- J1 pad 8: Net-(A1-5V) -> Net-(U2-GPIO15)
- J1 pad 9: Net-(A2-VS) -> Net-(U2-GPIO16)
- J2 pad 2: Net-(A1-GND) -> Net-(PS1--Vin)
- PS1 pad 1: Net-(A1-GND) -> Net-(PS1-+Vin)
- PS1 pad 2: unconnected-(PS1-NC-Pad2) -> Net-(PS1--Vin)
- PS1 pad 3: Net-(PS1-+Vin) -> Net-(Brd1-GND)
- PS1 pad 4: Net-(A1-GND) -> Net-(Brd1-VCC)
- Q1 pad 1: Net-(A1-GND) -> Net-(A2-GND)
- RDM1 pad GND: Net-(A1-GND) -> Net-(A2-GND)
- RDM1 pad RX: Net-(A1-GPIO10/SD3) -> Net-(Brd1-GND)
- SW1 pad 2: Net-(A1-GND) -> Net-(Brd1-GND)
- SW2 pad 2: Net-(A1-GND) -> Net-(Brd1-GND)
- SW3 pad 2: Net-(A1-GND) -> Net-(Brd1-GND)
- SW4 pad 2: Net-(A1-GND) -> Net-(Brd1-GND)
- U1 pad 3: Net-(A1-GND) -> Net-(PS1--Vin)
- U1 pad 4: Net-(A1-5V) -> Net-(Brd1-GND)
- U3 pad 1: Net-(A1-GND) -> unconnected-(U3-GND-Pad1)
- U3 pad 10: unconnected-(U3-GND-Pad10) -> Net-(A2-GND)
- U3 pad 5: Net-(A1-D5) -> Net-(U2-GPIO10_SS)
- U6 pad 1: Net-(A1-GND) -> Net-(A2-GND)
- U6 pad 8: Net-(A1-ADC1_CH5/D33) -> Net-(U2-GPIO10_SS)
Routing:
- net Net-(Brd1-GND): track 0.00 -> 417.8 mm, vias 0 -> 2
- net Net-(A1-GND): track 314.3 -> 0.00 mm
- net Net-(A2-GND): track 0.00 -> 153.0 mm, vias 0 -> 2
- net Net-(PS1--Vin): track 0.00 -> 130.2 mm, vias 0 -> 1
- net Net-(Brd1-VCC): track 0.00 -> 115.6 mm
- net Net-(U2-GPIO10_SS): track 0.00 -> 105.8 mm, vias 0 -> 1
- net Net-(Brd1-SCL): track 40.4 -> 120.2 mm, vias 0 -> 4
- net Net-(U2-GPIO17): track 0.00 -> 78.6 mm, vias 0 -> 1
- net Net-(U2-GPIO35): track 0.17 -> 75.8 mm, vias 0 -> 2
- net Net-(A1-ADC2_CH7/D27): track 73.8 -> 0.00 mm
- net Net-(U2-GPIO16): track 0.00 -> 73.2 mm, vias 0 -> 1
- net Net-(A1-ADC2_CH6/D14): track 73.1 -> 0.00 mm
- net Net-(A1-ADC2_CH4/D13): track 72.9 -> 0.00 mm
- net Net-(A1-GPIO10/SD3): track 67.5 -> 0.00 mm
- net Net-(A1-ADC1_CH5/D33): track 66.6 -> 0.00 mm
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Other:
- board text added: "${REFERENCE}"
- board text added: "Kraky debug board v2"
- board text removed: "Kraky debug board"
