File: kraky.kicad_sch (KiCad schematic)
At the start: 36 parts, among them J1 PINHD_1x10_Female, J2 JST_02, Q1 2N3904, SW1 Push_Button, SW2 Push_Button, SW3 Push_Button, SW4 Push_Button, SW5 SW_Nidec_CAS-120A1, U1 TP4056-42-ESOP8, U3 RFM98W-433S2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

Commit message: updated, read readme
Parts:
- added C5: 100nF, Capacitor_THT:C_Axial_L3.8mm_D2.6mm_P7.50mm_Horizontal, symbol Device:C
- added U4: MPU6050, PCM_SL_Breakout_Boards:MPU6050_Breakout, symbol PCM_SL_Breakout_Boards:MPU6050
- C1, C10, C2, C3, C4, C6, C7, C8: footprint Capacitor_SMD:C_0805_2012Metric -> Capacitor_THT:C_Axial_L3.8mm_D2.6mm_P7.50mm_Horizontal
- R1, R2, R3, R4, R5, R6, R9: footprint Resistor_SMD:R_0805_2012Metric_Pad1.20x1.40mm_HandSolder -> Resistor_THT:R_Axial_DIN0204_L3.6mm_D1.6mm_P5.08mm_Horizontal
Connections:
- net at A2.2 (GND), IRLED1.1 (C), Q1.1 (E)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: now also U4.7 (GND)
- net at BZ1.2, Brd1.1 (GND), C10.1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: now also C5.1
- net at A2.3 (VS), C4.1, C6.1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: now also C5.2, U4.8 (VCC)
- net at PS1.2 (NC): now also C10.2, C3.1, D1.1, J2.2, U1.3 (GND)
- net at Brd1.4 (SDA), U2.12 (GPIO08_SDA): now also U4.5 (SDA)
- net at Brd1.3 (SCL), U2.15 (GPIO09_SCL): now also U4.6 (SCL)
